File: cycle-7/cycle-7.kicad_pcb (KiCad board)
At the start: 2 copper layers, 347.7 x 94.2 mm, 176 parts, among them J1 Conn_01x06_MountingPin, J2 Conn_01x04_Pin, J3 Conn_01x02_Pin, SW1 SW_Push, U1 XC6206PxxxMR, U2 STM32F401RCTx, Y1 12MHz

Commit message: fixed layout, added gnd plane stitching
Parts:
- added U3: SRV05-4, PCM_marbastlib-various:SOT-23-6-routable, B.Cu at (233.5, 153.7)
- C1, C10, C11, C12, C13, C2, C3, C4, C5, C6, C7, C8, C9: footprint Capacitor_SMD:C_0402_1005Metric -> Capacitor_SMD:C_0603_1608Metric
- D74: footprint LED_SMD:LED_RGB_1210 -> lib-zegonix:SK6812MINI-E_3.2x2.8_reverse_mount; moved to B.Cu
- R1, R2, R3: footprint Resistor_SMD:R_0402_1005Metric -> Resistor_SMD:R_0603_1608Metric
- moved D74 9.44 mm to (375.6, 124.5), turned to 90 degrees
- moved C3 1.95 mm to (320.3, 126.0), turned to 135 degrees
- moved C13 1.62 mm to (326.3, 115.7)
- moved R3 1.42 mm to (329.4, 119.2)
- moved C6 1.41 mm to (335.9, 138.3)
- moved Y1 1.15 mm to (326.3, 119.2)
- moved R2 1.12 mm to (325.7, 141.4)
- moved R1 1.11 mm to (327.9, 141.4)
- moved C12 1.03 mm to (323.2, 119.2)
- moved C2 0.91 mm to (322.0, 124.3), turned to 135 degrees
- moved C11 0.42 mm to (337.3, 134.3)
Routing:
- net /LED_SIG: track 9.61 -> 53.3 mm, vias 0 -> 2
- net +3V3: track 159.7 -> 177.0 mm, vias 4 -> 6
- net GND: track 22.3 -> 31.6 mm, vias 1 -> 221
- net +5V: track 195.1 -> 199.6 mm
- net /COL14: track 225.9 -> 228.9 mm
- net /COL13: track 349.5 -> 352.5 mm
- net /COL15: track 198.0 -> 201.0 mm
- net /nRESET: track 62.0 -> 63.2 mm
- net /XIN: track 7.51 -> 8.69 mm
- net /COL4: track 289.3 -> 290.4 mm
- net /COL8: track 212.8 -> 214.0 mm
- net /COL7: track 248.1 -> 249.2 mm
- net /COL6: track 249.8 -> 251.0 mm
- net /COL5: track 291.3 -> 292.5 mm
- net /COL3: track 329.5 -> 330.7 mm
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
Commit message: added a kicad project for the plate added a kicad project for the daughter board
Routing:
- net /COL13: track 352.5 -> 351.5 mm
- net /USB_D+: track 161.3 -> 162.1 mm
- net GND: vias 221 -> 386

Commit message: implemented newest findings from prototype and updated to kicad 8
Parts:
- added R4: 10k, Resistor_SMD:R_0603_1608Metric, B.Cu at (345.6, 135.2)
- added R5: 10k, Resistor_SMD:R_0603_1608Metric, B.Cu at (306.1, 144.2)
- C11: value 100n -> 4.7u
Connections:
- J3 pad 1: /BOOTSEL -> +3V3
- J3 pad 2: GND -> /BOOT0
- U2 pad 28: unconnected-(U2-PB2-Pad28) -> /BOOT1
- U2 pad 60: /BOOTSEL -> /BOOT0
Routing:
- net /BOOT0: track 0.00 -> 35.1 mm, vias 0 -> 2
- net /BOOTSEL: track 27.9 -> 0.00 mm, vias 1 -> 0
- net /BOOT1: track 0.00 -> 15.4 mm, vias 0 -> 2
- net +3V3: track 177.0 -> 185.8 mm
- net GND: track 31.6 -> 30.4 mm, vias 386 -> 396
