File: daughter-board/daughter-board.kicad_sch (KiCad schematic)
At the start: 10 parts, among them J1 USB_C_Receptacle_USB2.0_16P, J2 Conn_01x06_MountingPin

Commit message: updated findings from prototype removed output folder as the vendors stock is everchanging
Parts:
- J2: footprint Connector_JST:JST_SHL_SM06B-SHLS-TF_1x06-1MP_P1.00mm_Horizontal -> Connector_JST:JST_SH_SM06B-SRSS-TB_1x06-1MP_P1.00mm_Horizontal
